File: esquematico_ESP32/esp32_2.kicad_sch (KiCad schematic)
At the start: 9 parts, among them U1 ESP32-WROOM-32

Commit message: placa terminada
Parts:
- Program1: renamed from Programador1; footprint Connector_PinSocket_2.54mm:PinSocket_1x05_P2.54mm_Horizontal -> Connector_PinSocket_2.54mm:PinSocket_1x05_P2.54mm_Vertical
Connections:
- net MAGNE_3: now also U1.27 (IO16); no longer U1.10 (IO25)
Other:
- sheet perifericos ports: added MAGNE_1; removed MAGNE_4
Changed lines of the file:
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@@
   (junction (at 132.08 66.04) (diameter 0) (color 0 0 0 0)
   )
+  (no_connect (at 236.22 102.87))
   (no_connect (at 205.74 64.77))
   (no_connect (at 205.74 67.31))
-  (no_connect (at 236.22 85.09))
   (no_connect (at 205.74 102.87))
   (no_connect (at 236.22 105.41))
@@
     (effects (font (size 1.27 1.27)) (justify left bottom))
   )
-  (label "MAGNE_3" (at 236.22 102.87 0)
+  (label "MAGNE_3" (at 236.22 85.09 0)
     (effects (font (size 1.27 1.27)) (justify left bottom))
   )
@@
     (effects (font (size 1.27 1.27)) (justify left bottom))
   )
-  (label "MAGNE_2" (at 87.63 82.55 0)
+  (label "MAGNE_2" (at 87.63 82.3976 0)
     (effects (font (size 1.27 1.27)) (justify left bottom))
   )
@@
     (effects (font (size 1.27 1.27)) (justify left bottom))
   )
-  (label "MAGNE_1" (at 87.63 80.01 0)
+  (label "MAGNE_1" (at 87.63 80.2894 0)
     (effects (font (size 1.27 1.27)) (justify left bottom))
   )
@@
     (effects (font (size 1.27 1.27)) (justify left bottom))
   )
-  (label "MAGNE_3" (at 87.63 85.09 0)
+  (label "MAGNE_3" (at 87.63 84.9376 0)
     (effects (font (size 1.27 1.27)) (justify left bottom))
   )
@@
   (symbol (lib_id "Connector:Conn_01x05_Female") (at 269.24 62.23 0) (mirror x) (unit 1)
     (in_bom yes) (on_board yes)
-    (property "Reference" "Programador1" (id 0) (at 262.89 71.12 0)
+    (property "Reference" "Program1" (id 0) (at 262.89 71.12 0)
       (effects (font (size 1.27 1.27)) (justify left))
     )
@@
       (effects (font (size 1.27 1.27)) (justify left))
     )
-    (property "Footprint" "Connector_PinSocket_2.54mm:PinSocket_1x05_P2.54mm_Horizontal" (id 2) (at 269.24 62.23 0)
+    (property "Footprint" "Connector_PinSocket_2.54mm:PinSocket_1x05_P2.54mm_Vertical" (id 2) (at 269.24 62.23 0)
       (effects (font (size 1.27 1.27)) hide)
     )
@@
       (effects (font (size 1.27 1.27)) (justify right))
     )
-    (pin "MAGNE_2" input (at 87.63 80.01 0)
-      (effects (font (size 1.27 1.27)) (justify right))
-    )
-    (pin "MAGNE_3" input (at 87.63 82.55 0)
-      (effects (font (size 1.27 1.27)) (justify right))
-    )
-    (pin "MAGNE_4" input (at 87.63 85.09 0)
+    (pin "MAGNE_2" input (at 87.63 82.3976 0)
+      (effects (font (size 1.27 1.27)) (justify right))
+    )
+    (pin "MAGNE_3" input (at 87.63 84.9376 0)
       (effects (font (size 1.27 1.27)) (justify right))
     )
@@
     (pin "CLC_KEY_3V3_ESP" input (at 36.83 74.93 180)
       (effects (font (size 1.27 1.27)) (justify left))
+    )
+    (pin "MAGNE_1" input (at 87.63 80.2894 0)
+      (effects (font (size 1.27 1.27)) (justify right))
     )
   )
@@
       (reference "C10") (unit 1) (value "220u") (footprint "Capacitor_SMD:CP_Elec_6.3x7.7")
     )
-    (path "/90dc18a7-d136-49c5-aca7-9f578dd2dde7/85341b1b-6741-403d-8334-5a36fd82bc82"
-      (reference "Conn_RFID1") (unit 1) (value "J2") (footprint "Connector_JST:JST_EH_S8B-EH_1x08_P2.50mm_Horizontal")
-    )
-    (path "/90dc18a7-d136-49c5-aca7-9f578dd2dde7/6f9cf025-6ba5-425e-926b-ef8018e09a41"
-      (reference "Conn_RFID2") (unit 1) (value "J3") (footprint "Connector_JST:JST_EH_S8B-EH_1x08_P2.50mm_Horizontal")
-    )
-    (path "/90dc18a7-d136-49c5-aca7-9f578dd2dde7/879dbbe4-ae64-435d-b735-afdb7f43184d"
-      (reference "Conn_screen1") (unit 1) (value "J5") (footprint "Connector_JST:JST_EH_S10B-EH_1x10_P2.50mm_Horizontal")
-    )
     (path "/90dc18a7-d136-49c5-aca7-9f578dd2dde7/7cbb4cf2-d39b-4cae-b2fd-23730c35b330"
       (reference "D1") (unit 1) (value "LED") (footprint "LED_SMD:LED_0805_2012Metric_Pad1.15x1.40mm_HandSolder")
@@
     )
     (path "/5125aeff-fbaf-4069-9b26-eba443c92f10/ab816942-ca37-4395-8381-87b62ed341fa/98c852c7-4008-4e0f-89ac-3d2c8aa0e3a2"
-      (reference "D4") (unit 1) (value "1N5825") (footprint "Diode_THT:D_DO-27_P12.70mm_Horizontal")
+      (reference "D4") (unit 1) (value "1N5825") (footprint "Diode_THT:D_DO-201AE_P5.08mm_Vertical_AnodeUp")
     )
     (path "/90dc18a7-d136-49c5-aca7-9f578dd2dde7/871fe201-8570-4ab4-b58c-0d248a209c25"
@@
     )
     (path "/5b1134d1-ab5f-48fa-b527-ffdc1b4c5ff5"
-      (reference "Programador1") (unit 1) (value "Conn_01x05_Female") (footprint "Connector_PinSocket_2.54mm:PinSocket_1x05_P2.54mm_Horizontal")
+      (reference "Program1") (unit 1) (value "Conn_01x05_Female") (footprint "Connector_PinSocket_2.54mm:PinSocket_1x05_P2.54mm_Vertical")
     )
     (path "/90dc18a7-d136-49c5-aca7-9f578dd2dde7/f793cc0c-ede8-43dc-9a01-a81d5ad3f9fc/698ef3e5-c802-45b7-80dd-701416eb8328"
@@
       (reference "R9") (unit 1) (value "10k") (footprint "Resistor_SMD:R_0805_2012Metric_Pad1.20x1.40mm_HandSolder")
     )
+    (path "/90dc18a7-d136-49c5-aca7-9f578dd2dde7/85341b1b-6741-403d-8334-5a36fd82bc82"
+      (reference "RFID1") (unit 1) (value "J2") (footprint "Connector_JST:JST_EH_S8B-EH_1x08_P2.50mm_Horizontal")
+    )
+    (path "/90dc18a7-d136-49c5-aca7-9f578dd2dde7/6f9cf025-6ba5-425e-926b-ef8018e09a41"
+      (reference "RFID2") (unit 1) (value "J3") (footprint "Connector_JST:JST_EH_S8B-EH_1x08_P2.50mm_Horizontal")
+    )
     (path "/7c72e10d-5c27-41ab-9844-8a388c7b7003"
       (reference "Rst1") (unit 1) (value "Enable") (footprint "Button_Switch_SMD:SW_SPST_CK_RS282G05A3")
@@
       (reference "Vin1") (unit 1) (value "Jack-DC") (footprint "Connector_BarrelJack:BarrelJack_Horizontal")
     )
-  )
+    (path "/90dc18a7-d136-49c5-aca7-9f578dd2dde7/879dbbe4-ae64-435d-b735-afdb7f43184d"
+      (reference "screen1") (unit 1) (value "J5") (footprint "Connector_JST:JST_EH_S10B-EH_1x10_P2.50mm_Horizontal")
+    )
+  )

Commit message: ajuste final
Connections:
- net D/C: now also U1.11 (IO26); no longer U1.7 (IO35)
- net RST_D: now also U1.10 (IO25); no longer U1.6 (IO34)
Changed lines of the file:
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@@
   (junction (at 132.08 66.04) (diameter 0) (color 0 0 0 0)
   )
-  (no_connect (at 236.22 102.87))
+  (no_connect (at 236.22 115.57))
+  (no_connect (at 236.22 118.11))
   (no_connect (at 205.74 64.77))
   (no_connect (at 205.74 67.31))
   (no_connect (at 205.74 102.87))
-  (no_connect (at 236.22 105.41))
   (no_connect (at 205.74 90.17))
   (no_connect (at 205.74 92.71))
@@
     (effects (font (size 1.27 1.27)) (justify right bottom))
   )
-  (label "D{slash}C" (at 236.22 118.11 0)
+  (label "D{slash}C" (at 236.22 105.41 0)
     (effects (font (size 1.27 1.27)) (justify left bottom))
   )
@@
     (effects (font (size 1.27 1.27)) (justify left bottom))
   )
-  (label "RST_D" (at 236.22 115.57 0)
-    (effects (font (size 1.27 1.27)) (justify left bottom))
-  )
+  (label "RST_D" (at 236.22 102.87 0)
+    (effects (font (size 1.27 1.27)) (justify left bottom))
+  )

Commit message: lista de materiales
Parts:
- C3: value 100u -> 100n
Changed lines of the file:
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@@
       (effects (font (size 1.27 1.27)) (justify left))
     )
-    (property "Value" "100u" (id 1) (at 195.58 46.99 0)
+    (property "Value" "100n" (id 1) (at 195.58 46.99 0)
       (effects (font (size 1.27 1.27)) (justify left))
     )
@@
     )
     (path "/0a8fb98b-26c6-43af-94b5-0a498a75c195"
-      (reference "C3") (unit 1) (value "100u") (footprint "Capacitor_SMD:C_0805_2012Metric_Pad1.18x1.45mm_HandSolder")
+      (reference "C3") (unit 1) (value "100n") (footprint "Capacitor_SMD:C_0805_2012Metric_Pad1.18x1.45mm_HandSolder")
     )
     (path "/5125aeff-fbaf-4069-9b26-eba443c92f10/47a92999-85b6-4838-bf9c-de8805710a0e"
