File: esquematico_ESP32/esp32_2.kicad_pcb (KiCad board)
At the start: 2 copper layers, 60 x 65 mm, 42 parts, among them Q1 BSS138, Q2 BSS138, T1 MountingHole_3.2mm_M3_DIN965, T2 MountingHole_3.2mm_M3_DIN965, T3 MountingHole_3.2mm_M3_DIN965, U1 ESP32-WROOM-32, U2 LM1117-3.3, U3 LM2596S-5

Commit message: ajuste final
Parts:
- moved T2 47.1 mm to (182.5, 30.5)
- moved T3 34.6 mm to (138.1, 46.5)
- moved T1 29.6 mm to (169.4, 57.1)
Connections:
- U1 pad 10: unconnected-(U1-Pad10) -> /RST_D
- U1 pad 11: unconnected-(U1-Pad11) -> /D/C
- U1 pad 6: /RST_D -> unconnected-(U1-Pad6)
- U1 pad 7: /D/C -> unconnected-(U1-Pad7)
Routing:
- net /RST_D: track 47.1 -> 42.0 mm
- net /D/C: track 48.9 -> 43.9 mm
